File: externalControls/External_Controls_Board.sch (EAGLE design)
At the start: 21 parts

Commit message: Rev1 Functional
updated to Rev1 specifications
Parts:
- removed DYNA1, DYNA2: DYNAMIXEL-1X03HORIZ, MRDT-2015-Arm:DYNAMIXEL-1X03HORIZ
- removed FET_DYNA1, FET_DYNA2, FET_DYNA3, FET_DYNA4, FET_DYNA5, FET_DYNA6: BUK9Y4R4-40EPOWER-SO8, MRDT-2015-General:BUK9Y4R4-40EPOWER-SO8
- removed LT1910CAP-DYNA1, LT1910CAP-DYNA2: .1µF, resistor:C-USC1206
- removed SV1: (no value), con-lsta:FE09W
- removed SV2, SV3: (no value), con-lsta:FE06W
- removed U$4: LT1910, MRDT-2015-PowerBoard:LT1910
- removed XB2: XBEE, maxstream:XBEE
- removed ZENER_DYNA1, ZENER_DYNA2: SMAJ5920, SparkFun-DiscreteSemi:DIODE-SCHOTTKY-MBRA140
- added U$8: MOLEX7-PIN, logicShifter:MOLEX7-PIN
- U$1: value LT1910 -> 74AHCT125; device MRDT-2015-PowerBoard:LT1910 -> logicShifter:74AHCT125
Connections:
- removed net 5V: FET_DYNA3.D, FET_DYNA4.D, FET_DYNA5.D, FET_DYNA6.D
- removed net CAM_12V: SV1.9, SV2.1
- removed net CAM_GND: SV1.8, SV2.2
- removed net CAM_PWM0: SV1.1, SV2.6
- removed net CAM_PWM1: SV1.2, SV2.5
- removed net CAM_PWM2: SV1.3, SV2.4
- removed net CAM_PWM3: SV1.4, SV2.3
- removed net CAM_VIDEO: SV1.7
- removed net CAM_VIDEO_GND: SV1.6
- removed net DYNA_ENABLE_1: U$2.PM4, U$4.IN
- removed net DYNA_ENABLE_2: U$1.IN, U$2.PM5
- removed net GATE-DYNA1: FET_DYNA1.G, U$4.GATE
- removed net GATE-DYNA2: FET_DYNA2.G, U$1.GATE
- removed net N: DYNA2.2, FET_DYNA2.S
- removed net NC: SV1.5
- removed net PWM0_OUT: SV3.1
- removed net PWM1_OUT: SV3.2
- removed net PWM2_OUT: SV3.3
- removed net PWM3_OUT: SV3.4
- removed net SOURCE-DYNA1: DYNA1.2, FET_DYNA1.S
- net +12V: now also U$8.P$2; no longer FET_DYNA1.D, FET_DYNA2.D, LT1910CAP-DYNA1.2, LT1910CAP-DYNA2.2, SV3.6, U$1.SENSE, U$1.V+, U$4.SENSE, U$4.V+
- net +5V: now also U$1.VCC
- net DYNA_DATA: now also U$8.P$3; no longer DYNA1.3, DYNA2.3, ZENER_DYNA1.C, ZENER_DYNA2.C
- net GND: now also U$1.1OE, U$1.2OE, U$1.3OE, U$1.4OE, U$8.P$1; no longer DYNA1.1, DYNA2.1, LT1910CAP-DYNA1.1, LT1910CAP-DYNA2.1, SV3.5, U$4.GND, ZENER_DYNA1.A, ZENER_DYNA2.A
- net N$1: now also U$1.1Y, U$8.P$7; no longer FET_DYNA3.S
- net N$2: now also U$1.2Y, U$8.P$6; no longer FET_DYNA4.S
- net N$3: now also U$1.3Y, U$8.P$5; no longer FET_DYNA5.S
- net N$4: now also U$1.4Y, U$8.P$4; no longer FET_DYNA6.S
- net TIVA_PWM0: now also U$1.1A; no longer FET_DYNA3.G
- net TIVA_PWM1: now also U$1.2A; no longer FET_DYNA4.G
- net TIVA_PWM2: now also U$1.3A; no longer FET_DYNA5.G
- net TIVA_PWM3: now also U$1.4A; no longer FET_DYNA6.G
Other:
- note removed: "these will be molex female 6 pin connectors"
